Commit message: New name motor joint

File: urdf/qube.macro.xacro (robot description, xacro)
@@ -1,4 +1,4 @@
 <?xml version="1.0"?>
-<robot xmlns:xacro="http://www.ros.org/wiki/xacro" name="qube_model">
+<robot xmlns:xacro="http://www.ros.org/wiki/xacro" name="qube">
   <!-- Define Properties for Flexibility -->
   <xacro:property name="stator_size" value="0.102 0.102 0.102"/>
@@ -7,5 +7,5 @@
   <xacro:property name="angle_size" value="0.025 0.002 0.002"/>
   <!-- Define the Macro with a single parameter "prefix" -->
-  <xacro:macro name="qube_model" params="prefix">
+  <xacro:macro name="qube" params="prefix">
     <!-- Links with prefixed names -->
     <link name="${prefix}_stator_link">
@@ -45,11 +45,19 @@
       <origin xyz="0 0 0.050" rpy="0 0 0"/>
     </joint>
-    <joint name="${prefix}_angle" type="revolute">
-      <parent link="${prefix}_stator_link"/>
-      <child link="${prefix}_rotor_link"/>
-      <origin xyz="0 0 0.05" rpy="0 0 0"/>
-      <limit lower="-3.14" upper="3.14" effort="10" velocity="1.0"/>
-      <axis xyz="0 0 1"/>
+<joint name="${prefix}_motor_joint" type="revolute">
+  <parent link="${prefix}_stator_link"/>
+  <child link="${prefix}_rotor_link"/>
+  <origin xyz="0 0 0.05" rpy="0 0 0"/>
+  <limit lower="-3.14" upper="3.14" effort="10" velocity="1.0"/>
+  <axis xyz="0 0 1"/>
+  <!-- Add ros2_control element below -->
+  <ros2_control name="${prefix}_motor_joint" type="transmission_interface/SimpleTransmission">
+    <joint name="${prefix}_motor_joint">
+      <command_interface name="velocity"/>
+      <state_interface name="velocity"/>
     </joint>
+    <actuator name="${prefix}_motor"/>
+  </ros2_control>
+</joint>
     <joint name="${prefix}_indicator" type="fixed">
       <parent link="${prefix}_rotor_link"/>

File: urdf/qube.urdf.xacro (robot description, xacro)
@@ -3,5 +3,5 @@
 	<xacro:include filename="$(find qube_description)/urdf/qube.macro.xacro" />
 	<link name="world"/>
-	<xacro:qube_model prefix="qube_model"/>
+	<xacro:qube prefix="qube"/>
 	<joint name="base_joint" type="fixed">
       <parent link="world"/>

Commit message: MOdified qube bringup so that the parameters for baudrate, device and simulation can be changed in the terminal

File: urdf/qube.macro.xacro (robot description, xacro)
@@ -9,5 +9,5 @@
   <xacro:macro name="qube" params="prefix">
     <!-- Links with prefixed names -->
-    <link name="${prefix}_stator_link">
+    <link name="${prefix}stator_link">
       <visual>
         <geometry>
@@ -19,5 +19,5 @@
       </visual>
     </link>
-    <link name="${prefix}_rotor_link">
+    <link name="${prefix}rotor_link">
       <visual>
         <geometry>
@@ -29,5 +29,5 @@
       </visual>
     </link>
-    <link name="${prefix}_angle_link">
+    <link name="${prefix}angle_link">
       <visual>
         <geometry>
@@ -40,27 +40,26 @@
     </link>
     <!-- Joints with prefixed names -->
-    <joint name="${prefix}_stator_joint" type="fixed">
+    <joint name="${prefix}stator_joint" type="fixed">
       <parent link="base_link"/>
-      <child link="${prefix}_stator_link"/>
+      <child link="${prefix}stator_link"/>
       <origin xyz="0 0 0.050" rpy="0 0 0"/>
     </joint>
-<joint name="${prefix}_motor_joint" type="revolute">
-  <parent link="${prefix}_stator_link"/>
-  <child link="${prefix}_rotor_link"/>
+<joint name="${prefix}motor_joint" type="continuous">
+  <parent link="${prefix}stator_link"/>
+  <child link="${prefix}rotor_link"/>
   <origin xyz="0 0 0.05" rpy="0 0 0"/>
-  <limit lower="-3.14" upper="3.14" effort="10" velocity="1.0"/>
   <axis xyz="0 0 1"/>
-  <!-- Add ros2_control element below -->
-  <ros2_control name="${prefix}_motor_joint" type="transmission_interface/SimpleTransmission">
-    <joint name="${prefix}_motor_joint">
-      <command_interface name="velocity"/>
-      <state_interface name="velocity"/>
-    </joint>
-    <actuator name="${prefix}_motor"/>
-  </ros2_control>
 </joint>
-    <joint name="${prefix}_indicator" type="fixed">
-      <parent link="${prefix}_rotor_link"/>
-      <child link="${prefix}_angle_link"/>
+    <!-- ros2_control transmission configuration -->
+    <ros2_control name="motor_joint" type="transmission_interface/SimpleTransmission">
+      <joint name="${prefix}motor_joint">
+        <command_interface name="velocity"/>
+        <state_interface name="velocity"/>
+        <state_interface name="position"/>
+      </joint>
+    </ros2_control>
+    <joint name="${prefix}indicator" type="fixed">
+      <parent link="${prefix}rotor_link"/>
+      <child link="${prefix}angle_link"/>
       <origin xyz="0.012 0 0.005" rpy="0 0 0"/>
     </joint>

File: urdf/qube.urdf.xacro (robot description, xacro)
@@ -3,5 +3,5 @@
 	<xacro:include filename="$(find qube_description)/urdf/qube.macro.xacro" />
 	<link name="world"/>
-	<xacro:qube prefix="qube"/>
+	<xacro:qube prefix="qube_"/>
 	<joint name="base_joint" type="fixed">
       <parent link="world"/>
